Commit message: initial commit

File: uuv_descriptions/urdf/rexrov.gazebo.xacro (robot description, xacro)
@@ -18,15 +18,15 @@
     assume NWU (otherwise cob is below cog?).
     -->
-    <xacro:property name="cob" value="0.0 0.0 0.3"/>
+    <xacro:property name="cob" value="0.0 0.0 0.05"/>
     <!-- Volume, see p.31 in Berg2012 -->
     <xacro:property name="volume" value="1.83826"/>
     <xacro:macro name="rexrov_hydro_model" params="namespace">
         <link name="${namespace}/base_link">
-            <neutrally_buoyant>0</neutrally_buoyant>
+            <neutrally_buoyant>1</neutrally_buoyant>
             <volume>${volume}</volume>
             <box>
-                <width>1.5</width>
-                <length>2.6</length>
-                <height>1.6</height>
+                <width>0.5</width>
+                <length>1.0</length>
+                <height>0.4</height>
             </box>
             <center_of_buoyancy>${cob}</center_of_buoyancy>

File: uuv_descriptions/urdf/rexrov_actuators.xacro (robot description, xacro)
@@ -26,27 +26,35 @@
     </xacro:thruster_module_first_order_basic_fcn_macro>
   </xacro:macro>
-  <xacro:thruster_macro namespace="${namespace}" thruster_id="0">
-    <origin xyz="-0.890895 0.334385 0.528822" rpy="${0*d2r} ${-74.53*d2r} ${-53.21*d2r}"/>
+    <xacro:thruster_macro namespace="${namespace}" thruster_id="0">
+    <!-- <East> -->
+    <origin xyz="-0.00295 0.155242 -0.256919" rpy="0 0.00 0" />
   </xacro:thruster_macro>
   <xacro:thruster_macro namespace="${namespace}" thruster_id="1">
-    <origin xyz="-0.890895 -0.334385 0.528822" rpy="${0*d2r} ${-74.53*d2r} ${53.21*d2r}"/>
+    <!-- <West> -->
+    <origin xyz="-0.00294 -0.223659 -0.256867" rpy="0 0.00 0" />
   </xacro:thruster_macro>
   <xacro:thruster_macro namespace="${namespace}" thruster_id="2">
-    <origin xyz="0.890895 0.334385 0.528822" rpy="${0*d2r} ${-105.47*d2r} ${53.21*d2r}"/>
+    <!-- <North> -->
+    <origin xyz="-0.349097 -0.02119 -0.259973" rpy="0 0 1.5708" />
   </xacro:thruster_macro>
   <xacro:thruster_macro namespace="${namespace}" thruster_id="3">
-    <origin xyz="0.890895 -0.334385 0.528822" rpy="${0*d2r} ${-105.47*d2r} ${-53.21*d2r}"/>
+    <!-- <South> -->
+    <origin xyz="0.469063 -0.02119 -0.253872" rpy="0 0 1.5708" />
   </xacro:thruster_macro>
   <xacro:thruster_macro namespace="${namespace}" thruster_id="4">
-    <origin xyz="-0.412125 0.505415 0.129" rpy="${0*d2r} ${0*d2r} ${45*d2r}"/>
+    <!-- <South-West> -->
+    <origin xyz="0.449063 -0.203659 -0.256919" rpy="0 -1.5708 0" />
   </xacro:thruster_macro>
   <xacro:thruster_macro namespace="${namespace}" thruster_id="5">
-    <origin xyz="-0.412125 -0.505415 0.129" rpy="${0*d2r} ${0*d2r} ${-45*d2r}"/>
+    <!-- <North-West> -->
+    <origin xyz="-0.319097 -0.203659 -0.256919" rpy="0 -1.5708 0" />
   </xacro:thruster_macro>
   <xacro:thruster_macro namespace="${namespace}" thruster_id="6">
-    <origin xyz="0.412125 0.505415 0.129" rpy="${0*d2r} ${0*d2r} ${135*d2r}"/>
+    <!-- <North-East> -->
+    <origin xyz="-0.319078 0.135242 -0.256919" rpy="0 -1.5708 0" />
   </xacro:thruster_macro>
   <xacro:thruster_macro namespace="${namespace}" thruster_id="7">
-    <origin xyz="0.412125 -0.505415 0.129" rpy="${0*d2r} ${0*d2r} ${-135*d2r}"/>
+    <!-- <South-East> -->
+    <origin xyz="0.449034 0.135242 -0.256919" rpy=" 0 -1.5708 0" />
   </xacro:thruster_macro>
 </robot>

File: uuv_descriptions/urdf/rexrov_base.xacro (robot description, xacro)
@@ -27,8 +27,9 @@
   <!-- Parameters -->
   <xacro:property name="namespace" value="rexrov"/>
-  <xacro:property name="visual_mesh_file" value="file://$(find uuv_descriptions)/meshes/RexROV_no_props.dae"/>
+  <xacro:property name="visual_mesh_file" value="file://$(find uuv_descriptions)/meshes/vehicle.STL"/>
   <xacro:property name="prop_mesh_file" value="file://$(find uuv_descriptions)/meshes/prop.dae"/>
+  <xacro:property name="collision_mesh_file" value="file://$(find uuv_descriptions)/meshes/vehicle.STL"/>
   <!-- Mass, see p.28 in Berg2012 -->
-  <xacro:property name="mass" value="1862.87"/>
+  <xacro:property name="mass" value="862.87"/>
   <xacro:macro name="rexrov_base" params="namespace *gazebo inertial_reference_frame">
     <!-- base_link according to ROS conventions: x forward, z up -->
@@ -37,5 +38,5 @@
         <mass value="${mass}"/>
         <origin xyz="0 0 0"/>
-        <inertia ixx="525.39" ixy="1.44" ixz="33.41" iyy="794.20" iyz="2.6" izz="691.23"/>
+        <inertia ixx="243.39" ixy="1.44" ixz="33.41" iyy="367.20" iyz="2.6" izz="319.23"/>
       </inertial>
       <visual>
@@ -45,24 +46,9 @@
         </geometry>
       </visual>
-      <!-- bottom plate -->
       <collision>
-        <origin xyz="0 0 -0.75" rpy="0 0 0"/>
+        <origin xyz="0 0 0" rpy="0 0 0"/>
         <geometry>
-          <box size="2.56 1.50 0.10"/>
+          <mesh filename="${collision_mesh_file}" scale="1 1 1" />
         </geometry>
-      </collision>
-      <!-- top plate -->
-      <collision>
-        <origin xyz="0 0 0.60" rpy="0 0 0"/>
-        <geometry><box size="2.56 1.50 0.40"/></geometry>
-      </collision>
-      <!-- left / right sides -->
-      <collision>
-        <origin xyz="-0.20 0.70 -0.15" rpy="0 0 0"/>
-        <geometry><box size="2.20 0.10 1.10"/></geometry>
-      </collision>
-      <collision>
-        <origin xyz="-0.20 -0.70 -0.15" rpy="0 0 0"/>
-        <geometry><box size="2.20 0.10 1.10"/></geometry>
       </collision>
     </link>

File: uuv_descriptions/urdf/rexrov_sensors.xacro (robot description, xacro)
@@ -13,20 +13,14 @@
 -->
 <robot xmlns:xacro="http://www.ros.org/wiki/xacro">
-  <!-- DVL  -->
+  <!-- DVL -->
   <xacro:default_dvl_macro
     namespace="${namespace}"
     parent_link="${namespace}/base_link"
     inertial_reference_frame="${inertial_reference_frame}">
-    <origin xyz="-1.4 0 -0.312" rpy="0 ${0.5*pi} 0"/>
+    <origin xyz="-0.219097 -0.04 -0.312" rpy="0 ${0.5*pi} 0"/>
   </xacro:default_dvl_macro>
-  <!-- Magnetometer  -->
-  <xacro:default_magnetometer namespace="${namespace}" parent_link="${namespace}/base_link"/>
-  <!-- RPT  -->
-  <xacro:default_rpt namespace="${namespace}" parent_link="${namespace}/base_link">
-    <origin xyz="-1.32 0 0.8" rpy="0 0 0"/>
-  </xacro:default_rpt>
   <!-- Pressure  -->
   <xacro:default_pressure_macro namespace="${namespace}" parent_link="${namespace}/base_link">
-    <origin xyz="-1.32 0.5 0.85" rpy="0 0 0"/>
+    <origin xyz="0 0 -0.370" rpy="0 0 0"/>
   </xacro:default_pressure_macro>
   <!-- IMU  -->
@@ -37,20 +31,9 @@
     <origin xyz="0 0 0" rpy="0 0 0"/>
   </xacro:default_imu_macro>
-  <!-- Mount a camera -->
-  <xacro:default_camera namespace="${namespace}" parent_link="${namespace}/base_link" suffix="">
-    <origin xyz="1.15 0 0.4" rpy="0 0.6 0"/>
+  <xacro:default_camera namespace="${namespace}" parent_link="${namespace}/base_link" suffix="front">
+    <origin xyz="0.459063 -0.02119 -0.1724" rpy="0 0 0"/>
   </xacro:default_camera>
-  <xacro:default_camera namespace="${namespace}" parent_link="${namespace}/base_link" suffix="right">
-    <origin xyz="1.15 -0.63 0.4" rpy="0 0.6 0.4"/>
+  <xacro:default_camera namespace="${namespace}" parent_link="${namespace}/base_link" suffix="bottom">
+    <origin xyz="0.049983 -0.02119 -0.379224" rpy="0 1.7142 0"/>
   </xacro:default_camera>
-  <xacro:default_camera namespace="${namespace}" parent_link="${namespace}/base_link" suffix="left">
-    <origin xyz="1.15 0.63 0.4" rpy="0 0.6 -0.4"/>
-  </xacro:default_camera>
-  <!-- Mount a GPS. -->
-  <xacro:default_gps namespace="${namespace}" parent_link="${namespace}/base_link" />
-  <!-- Mount a Pose 3D sensor. -->
-  <xacro:default_pose_3d_macro
-    namespace="${namespace}"
-    parent_link="${namespace}/base_link"
-    inertial_reference_frame="${inertial_reference_frame}" />
 </robot>

File: uuv_gazebo_plugins/uuv_gazebo_ros_plugins/urdf/thruster_snippets.xacro (robot description, xacro)
@@ -89,5 +89,5 @@
         <origin rpy="0 0 0" xyz="0 0 0"/>
         <geometry>
-          <mesh filename="${mesh_filename}" scale="1 1 1"/>
+          <mesh filename="${mesh_filename}" scale="0.25 0.25 0.25"/>
         </geometry>
       </visual>

File: uuv_sensor_plugins/uuv_sensor_ros_plugins/urdf/dvl_snippets.xacro (robot description, xacro)
@@ -31,5 +31,5 @@
       noise_sigma="0"
       noise_amplitude="0"
-      scale="1">
+      scale="0.4">
       <xacro:insert_block name="origin" />
     </xacro:dvl_plugin_macro>
