Commit message: added stereo cameras

File: anahita_description/urdf/anahita_sensors.xacro (robot description, xacro)
@@ -31,7 +31,15 @@
     <origin xyz="0 0 0" rpy="0 0 0"/>
   </xacro:default_imu_macro>
+  <!-- Stereo -->
+  <xacro:duo3d_camera
+    namespace="${namespace}"
+    parent_link="${namespace}/base_link">
+    <origin xyz="0.459063 -0.02119 -0.1124" rpy="0 0 0" />
+  </xacro:duo3d_camera>
+  <!-- Front Camera -->
   <xacro:default_camera namespace="${namespace}" parent_link="${namespace}/base_link" suffix="front">
     <origin xyz="0.459063 -0.02119 -0.1724" rpy="0 0 0"/>
   </xacro:default_camera>
+  <!-- Bottom Camera -->
   <xacro:default_camera namespace="${namespace}" parent_link="${namespace}/base_link" suffix="bottom">
     <origin xyz="0.049983 -0.02119 -0.379224" rpy="0 1.5714285714 0"/>

File: uuv_sensor_plugins/uuv_sensor_ros_plugins/urdf/stereo_snippets.xacro (robot description, xacro)
@@ -23,5 +23,5 @@
   <xacro:property name="p2r" value="0.002447"/>
   <xacro:property name="k3r" value="0.000000"/>
-  <xacro:property name="hfov" value="1.3844"/>
+  <xacro:property name="hfov" value="1.047198"/>
   <!-- Macro for a minimal collision block (for when you do not want collision block but gazebo needs one) -->
   <xacro:macro name="no_collision">
@@ -34,5 +34,5 @@
   </xacro:macro>
   <xacro:macro name="duo3d_camera" params="namespace parent_link *origin">
-    <link name="${namespace}/duo3d_left_link">
+    <link name="${namespace}/duo3d_link">
       <inertial>
         <mass value="0.01"/>
@@ -49,10 +49,10 @@
       <xacro:insert_block name="origin" />
       <parent link="${parent_link}" />
-      <child link="${namespace}/duo3d_left_link" />
+      <child link="${namespace}/duo3d_link" />
       <limit upper="0" lower="0" effort="0" velocity="0" />
       <axis xyz="1 0 0"/>
     </joint>
-    <gazebo reference="${namespace}/duo3d_left_link">
-      <sensor name="camera" type="camera">
+    <gazebo reference="${namespace}/duo3d_link">
+      <sensor name="camera" type="depth">
       <camera>
         <horizontal_fov>${hfov}</horizontal_fov>
@@ -64,23 +64,21 @@
         <clip>
           <near>0.05</near>
-          <far>5000</far>
+          <far>8</far>
         </clip>
-        <distortion>
-          <k1>${k1l}</k1>
-          <k2>${k2l}</k2>
-          <k3>${k3l}</k3>
-          <p1>${p1l}</p1>
-          <p2>${p2l}</p2>
-          <center>0.5 0.5</center>
-        </distortion>
       </camera>
-      <plugin name="left_controller" filename="libgazebo_ros_camera.so">
+      <plugin name="camera_plugin" filename="libgazebo_ros_openni_kinect.so">
+        <baseline>0.2</baseline>
         <alwaysOn>true</alwaysOn>
-        <updateRate>30.0</updateRate>
-        <cameraName>${namespace}/duo3d_left</cameraName>
-        <imageTopicName>image_raw</imageTopicName>
-        <cameraInfoTopicName>camera_info</cameraInfoTopicName>
-        <frameName>${namespace}/duo3d_left_link</frameName>
-        <hackBaseline>0.07</hackBaseline>
+        <!-- Keep this zero, update_rate in the parent <sensor> tag
+          will control the frame rate. -->
+        <updateRate>0</updateRate>
+        <cameraName>camera_ir</cameraName>
+        <imageTopicName>/camera/color/image_raw</imageTopicName>
+        <cameraInfoTopicName>/camera/depth/camera_info</cameraInfoTopicName>
+        <depthImageTopicName>/camera/depth/image_raw</depthImageTopicName>
+        <depthImageInfoTopicName>/camera/depth/camera_info</depthImageInfoTopicName>
+        <pointCloudTopicName>/camera/depth/points</pointCloudTopicName>
+        <frameName>camera_link</frameName>
+        <pointCloudCutoff>0.05</pointCloudCutoff>
         <distortionK1>${k1l}</distortionK1>
         <distortionK2>${k2l}</distortionK2>
@@ -88,4 +86,9 @@
         <distortionT1>${p1l}</distortionT1>
         <distortionT2>${p2l}</distortionT2>
+        <CxPrime>0</CxPrime>
+        <Cx>0</Cx>
+        <Cy>0</Cy>
+        <focalLength>0</focalLength>
+        <hackBaseline>0</hackBaseline>
       </plugin>
       <always_on>1</always_on>
@@ -94,59 +97,4 @@
     </sensor>
     </gazebo>
-    <link name="${namespace}/duo3d_right_link">
-      <inertial>
-        <mass value="0.01"/>
-        <inertia ixx="0" ixy="0.0" ixz="0.0" iyy="0" iyz="0.0" izz="0" />
-      </inertial>
-      <xacro:no_collision/>
-    </link>
-    <joint name="${namespace}/duo3d_right_joint" type="revolute">
-      <origin xyz="0.0 -0.03 0" rpy="0 0 0"/>
-      <parent link="${namespace}/duo3d_left_link" />
-      <child link="${namespace}/duo3d_right_link" />
-      <limit upper="0" lower="0" effort="0" velocity="0" />
-      <axis xyz="1 0 0"/>
-    </joint>
-    <gazebo reference="${namespace}/duo3d_right_link">
-      <sensor name="camera" type="camera">
-      <camera>
-        <horizontal_fov>${hfov}</horizontal_fov>
-        <image>
-          <width>640</width>
-          <height>460</height>
-          <format>R8G8B8</format>
-        </image>
-        <clip>
-          <near>0.05</near>
-          <far>5000</far>
-        </clip>
-        <distortion>
-          <k1>${k1l}</k1>
-          <k2>${k2l}</k2>
-          <k3>${k3l}</k3>
-          <p1>${p1l}</p1>
-          <p2>${p2l}</p2>
-          <center>0.5 0.5</center>
-        </distortion>
-      </camera>
-      <plugin name="right_controller" filename="libgazebo_ros_camera.so">
-        <alwaysOn>true</alwaysOn>
-        <updateRate>30.0</updateRate>
-        <cameraName>${namespace}/duo3d_right</cameraName>
-        <imageTopicName>image_raw</imageTopicName>
-        <cameraInfoTopicName>camera_info</cameraInfoTopicName>
-        <frameName>${namespace}/duo3d_right_link</frameName>
-        <hackBaseline>0.07</hackBaseline>
-        <distortionK1>${k1l}</distortionK1>
-        <distortionK2>${k2l}</distortionK2>
-        <distortionK3>${k3l}</distortionK3>
-        <distortionT1>${p1l}</distortionT1>
-        <distortionT2>${p2l}</distortionT2>
-      </plugin>
-      <always_on>1</always_on>
-      <update_rate>30</update_rate>
-      <visualize>true</visualize>
-    </sensor>
-  </gazebo>
   </xacro:macro>
 </robot>
