Commit message: implemented dynamic model of anahita

File: anahita_description/urdf/anahita_base.xacro (robot description, xacro)
@@ -31,5 +31,9 @@
   <xacro:property name="collision_mesh_file" value="file://$(find anahita_description)/meshes/vehicle.STL"/>
   <!-- Mass, see p.28 in Berg2012 -->
-  <xacro:property name="mass" value="862.87"/>
+  <xacro:property name="mass" value="35"/>
+  <xacro:property name="x_size" value="0.88"/>
+  <xacro:property name="y_size" value="0.40"/>
+  <xacro:property name="z_size" value="0.35"/>
+  <xacro:property name="equivalent_radius" value="${0.5*z_size}"/>
   <xacro:macro name="anahita_base" params="namespace *gazebo inertial_reference_frame">
     <!-- base_link according to ROS conventions: x forward, z up -->
@@ -38,5 +42,7 @@
         <mass value="${mass}"/>
         <origin xyz="0 0 0"/>
-        <inertia ixx="243.39" ixy="1.44" ixz="33.41" iyy="367.20" iyz="2.6" izz="319.23"/>
+        <inertia ixx="${0.2*mass*y_size*y_size + 0.2*mass*z_size*z_size}" ixy="0.0" ixz="0.0"
+               iyy="${0.2*mass*x_size*x_size + 0.2*mass*z_size*z_size}" iyz="0.0"
+               izz="${0.2*mass*x_size*x_size + 0.2*mass*y_size*y_size}" />
       </inertial>
       <visual>

File: anahita_description/urdf/anahita_gazebo.xacro (robot description, xacro)
@@ -20,5 +20,5 @@
     <xacro:property name="cob" value="0.0 0.0 0.05"/>
     <!-- Volume, see p.31 in Berg2012 -->
-    <xacro:property name="volume" value="0.5"/>
+    <xacro:property name="volume" value="0.2"/>
     <xacro:macro name="anahita_hydro_model" params="namespace">
         <link name="${namespace}/base_link">
@@ -27,5 +27,5 @@
             <box>
                 <width>0.5</width>
-                <length>1.0</length>
+                <length>0.88</length>
                 <height>0.4</height>
             </box>
@@ -35,18 +35,18 @@
                 <!-- Added mass: see p.28 in Berg2012 -->
                 <added_mass>
-                     779.79 -6.8773 -103.32  8.5426 -165.54 -7.8033
-                    -6.8773    1222   51.29  409.44 -5.8488  62.726
-                    -103.32   51.29  3659.9  6.1112 -386.42  10.774
-                     8.5426  409.44  6.1112   534.9 -10.027  21.019
-                    -165.54 -5.8488 -386.42 -10.027  842.69 -1.1162
-                    -7.8033  62.726  10.775  21.019 -1.1162  224.32
+                    1.7182 0 0 0 0 0
+                    0 0 0 0 0 0
+                    0 0 5.468 0 0 0
+                    0 0 0 0 0 0
+                    0 0 0 0 1.2481 0
+                    0 0 0 0 0 0.4006
                 </added_mass>
                 <!-- Linear damping: see p.31 in Berg2012 -->
                 <linear_damping>
-                    -74.82 -69.48 -728.4 -268.8 -309.77 -105
+                    -11.7391 -20 -31.8678 -25 -44.9085 -5
                 </linear_damping>
                 <!-- Non-linear damping: see p.30 in Berg2012 -->
                 <quadratic_damping>
-                    -748.22 -992.53 -1821.01 -672 -774.44 -523.27
+                    0 0 0 0 0 0
                 </quadratic_damping>
             </hydrodynamic_model>
