Commit message: modified stereo xacro

File: uuv_sensor_plugins/uuv_sensor_ros_plugins/urdf/pressure_snippets.xacro (robot description, xacro)
@@ -36,5 +36,5 @@
       kPaPerM="9.80638">
       <inertia ixx="0.00001" ixy="0.0" ixz="0.0" iyy="0.00001" iyz="0.0" izz="0.00001" />
-      <xacro:insert_block name="origin" />>
+      <xacro:insert_block name="origin" />
     </xacro:pressure_plugin_macro>
   </xacro:macro>
@@ -69,5 +69,5 @@
       <visual>
         <geometry>
-          <mesh filename="file://$(find uuv_sensor_ros_plugins)/meshes/pressure.dae" scale="1 1 1"/>
+          <mesh filename="file://$(find uuv_sensor_ros_plugins)/meshes/pressure.dae" scale="0.25 0.25 0.25"/>
         </geometry>
       </visual>

File: uuv_sensor_plugins/uuv_sensor_ros_plugins/urdf/stereo_snippets.xacro (robot description, xacro)
@@ -23,5 +23,5 @@
   <xacro:property name="p2r" value="0.002447"/>
   <xacro:property name="k3r" value="0.000000"/>
-  <xacro:property name="hfov" value="1.047198"/>
+  <xacro:property name="hfov" value="1.512198"/>
   <!-- Macro for a minimal collision block (for when you do not want collision block but gazebo needs one) -->
   <xacro:macro name="no_collision">
@@ -33,5 +33,5 @@
     </collision>
   </xacro:macro>
-  <xacro:macro name="duo3d_camera" params="namespace parent_link *origin">
+  <xacro:macro name="duo3d_camera_depth" params="namespace parent_link *origin">
     <link name="${namespace}/duo3d_link">
       <inertial>
@@ -58,6 +58,6 @@
         <horizontal_fov>${hfov}</horizontal_fov>
         <image>
-          <width>640</width>
-          <height>460</height>
+          <width>768</width>
+          <height>492</height>
           <format>R8G8B8</format>
         </image>
@@ -98,3 +98,120 @@
     </gazebo>
   </xacro:macro>
+  <xacro:macro name="duo3d_camera" params="namespace parent_link *origin">
+    <link name="${namespace}/duo3d_left_link">
+      <inertial>
+        <mass value="0.01"/>
+        <inertia ixx="0" ixy="0.0" ixz="0.0" iyy="0" iyz="0.0" izz="0" />
+      </inertial>
+      <visual>
+        <geometry>
+          <mesh filename="file://$(find uuv_sensor_ros_plugins)/meshes/duo3d.dae"/>
+        </geometry>
+      </visual>
+      <xacro:no_collision/>
+    </link>
+    <joint name="${namespace}/duo3d_joint" type="revolute">
+      <xacro:insert_block name="origin" />
+      <parent link="${parent_link}" />
+      <child link="${namespace}/duo3d_left_link" />
+      <limit upper="0" lower="0" effort="0" velocity="0" />
+      <axis xyz="1 0 0"/>
+    </joint>
+    <gazebo reference="${namespace}/duo3d_left_link">
+      <sensor name="camera" type="camera">
+      <camera>
+        <horizontal_fov>${hfov}</horizontal_fov>
+        <image>
+          <width>768</width>
+          <height>492</height>
+          <format>R8G8B8</format>
+        </image>
+        <clip>
+          <near>0.05</near>
+          <far>5000</far>
+        </clip>
+        <distortion>
+          <k1>${k1l}</k1>
+          <k2>${k2l}</k2>
+          <k3>${k3l}</k3>
+          <p1>${p1l}</p1>
+          <p2>${p2l}</p2>
+          <center>0.5 0.5</center>
+        </distortion>
+      </camera>
+      <plugin name="left_controller" filename="libgazebo_ros_camera.so">
+        <alwaysOn>true</alwaysOn>
+        <updateRate>30.0</updateRate>
+        <cameraName>left</cameraName>
+        <imageTopicName>image_raw</imageTopicName>
+        <cameraInfoTopicName>camera_info</cameraInfoTopicName>
+        <frameName>${namespace}/duo3d_left_link</frameName>
+        <hackBaseline>0.07</hackBaseline>
+        <distortionK1>${k1l}</distortionK1>
+        <distortionK2>${k2l}</distortionK2>
+        <distortionK3>${k3l}</distortionK3>
+        <distortionT1>${p1l}</distortionT1>
+        <distortionT2>${p2l}</distortionT2>
+      </plugin>
+      <always_on>1</always_on>
+      <update_rate>30</update_rate>
+      <visualize>true</visualize>
+    </sensor>
+    </gazebo>
+    <link name="${namespace}/duo3d_right_link">
+      <inertial>
+        <mass value="0.01"/>
+        <inertia ixx="0" ixy="0.0" ixz="0.0" iyy="0" iyz="0.0" izz="0" />
+      </inertial>
+      <xacro:no_collision/>
+    </link>
+    <joint name="${namespace}/duo3d_right_joint" type="revolute">
+      <origin xyz="0.0 -0.03 0" rpy="0 0 0"/>
+      <parent link="${namespace}/duo3d_left_link" />
+      <child link="${namespace}/duo3d_right_link" />
+      <limit upper="0" lower="0" effort="0" velocity="0" />
+      <axis xyz="1 0 0"/>
+    </joint>
+    <gazebo reference="${namespace}/duo3d_right_link">
+      <sensor name="camera" type="camera">
+      <camera>
+        <horizontal_fov>${hfov}</horizontal_fov>
+        <image>
+          <width>768</width>
+          <height>492</height>
+          <format>R8G8B8</format>
+        </image>
+        <clip>
+          <near>0.05</near>
+          <far>5000</far>
+        </clip>
+        <distortion>
+          <k1>${k1l}</k1>
+          <k2>${k2l}</k2>
+          <k3>${k3l}</k3>
+          <p1>${p1l}</p1>
+          <p2>${p2l}</p2>
+          <center>0.5 0.5</center>
+        </distortion>
+      </camera>
+      <plugin name="right_controller" filename="libgazebo_ros_camera.so">
+        <alwaysOn>true</alwaysOn>
+        <updateRate>30.0</updateRate>
+        <cameraName>right</cameraName>
+        <imageTopicName>image_raw</imageTopicName>
+        <cameraInfoTopicName>camera_info</cameraInfoTopicName>
+        <frameName>${namespace}/duo3d_right_link</frameName>
+        <hackBaseline>0.07</hackBaseline>
+        <distortionK1>${k1l}</distortionK1>
+        <distortionK2>${k2l}</distortionK2>
+        <distortionK3>${k3l}</distortionK3>
+        <distortionT1>${p1l}</distortionT1>
+        <distortionT2>${p2l}</distortionT2>
+      </plugin>
+      <always_on>1</always_on>
+      <update_rate>30</update_rate>
+      <visualize>true</visualize>
+    </sensor>
+  </gazebo>
+  </xacro:macro>
 </robot>
