Commit message: minor fixes

File: uuv_gazebo_worlds/models/StartGate/StartGate.xacro (robot description, xacro)
@@ -26,5 +26,5 @@
         rpy="0 0 0" />
       <geometry>
-        <mesh filename="package://robosub_descriptions/models/StartGate/StartGate.dae" />
+        <mesh filename="package://uuv_gazebo_worlds/models/StartGate/StartGate.dae" />
       </geometry>
     </visual>
@@ -34,5 +34,5 @@
         rpy="0 0 0" />
       <geometry>
-        <mesh filename="package://robosub_descriptions/models/StartGate/StartGate.dae" />
+        <mesh filename="package://uuv_gazebo_worlds/models/StartGate/StartGate.dae" />
       </geometry>
     </collision>

File: uuv_gazebo_worlds/models/Torpedo/Torpedo.xacro (robot description, xacro)
@@ -24,5 +24,5 @@
       <geometry>
         <mesh
-          filename="package://robosub_descriptions/models/Torpedo/Torpedo.stl" />
+          filename="package://uuv_gazebo_worlds/models/Torpedo/Torpedo.stl" />
       </geometry>
     </visual>
@@ -33,5 +33,5 @@
       <geometry>
         <mesh
-          filename="package://robosub_descriptions/models/Torpedo/Torpedo.stl" />
+          filename="package://uuv_gazebo_worlds/models/Torpedo/Torpedo.stl" />
       </geometry>
     </collision>

Commit message: Added several things

File: uuv_gazebo_worlds/models/StartGate/StartGate.xacro (robot description, xacro)
@@ -4,5 +4,5 @@
 <!-- Loading file with sensor macros -->
 <xacro:include filename="$(find uuv_sensor_ros_plugins)/urdf/sensor_snippets.xacro"/>
-<xacro:macro name="startgate_base" params="namespace">
+<xacro:macro name="startgate_base">
   <link
     name="${namespace}/base_link">
