Commit message: fixed triangular buoy

File: uuv_gazebo_worlds/models/Buoy_Akash/urdf/Buoy_Akash.urdf (robot description, URDF)
Before this commit: robot Buoy_Akash, 4 links, 3 joints
Links:
- link Board_1: mass 8.9187 -> 2.2297
- link Board_2: mass 8.9187 -> 2.2297
- link Board_3: mass 8.9187 -> 2.2297
- link base_link: mass 7.86706899154168 -> 0.98338

Commit message: fixed mass for collision with bot

File: uuv_gazebo_worlds/models/Buoy_Akash/urdf/Buoy_Akash.urdf (robot description, URDF)
Before this commit: robot Buoy_Akash, 4 links, 3 joints
Links:
- link base_link: mass 0.98338 -> 100000
